Commit message: add new model

File: urdf/blue_box.urdf (robot description, URDF)
Before this commit: robot conveyor_belt, 2 links, 1 joints
Links:
- removed link world
Joints:
- removed joint joint_fix

File: urdf/red_cylinder.urdf (robot description, URDF)
Before this commit: robot conveyor_belt, 2 links, 1 joints
Links:
- removed link world
Joints:
- removed joint joint_fix
