Commit message: update scara robot model

File: urdf/scara_robot_left.urdf (robot description, URDF)
Before this commit: robot scara_robot, 9 links, 8 joints
Links:
- link arm1: geometry collision box size=0.1 1.1 0.1; visual box size=0.1 1.1 0.1
- link arm2: geometry collision box size=0.1 0.9 0.1; visual box size=0.1 0.9 0.1
Joints:
- joint finger1_joint: axis 1 0 0 -> 0 1 0; limit lower=-0.01 upper=0.0 effort=100 velocity=100 -> lower=0.0 upper=0.01 effort=100 velocity=100; origin xyz=0.03 0 -0.23 rpy=0 0 0 -> xyz=0 -0.03 -0.23 rpy=0 0 0
- joint finger2_joint: axis 0 1 0 -> 1 0 0; origin xyz=0 0.03 -0.23 rpy=0 0 0 -> xyz=0.03 0 -0.23 rpy=0 0 0
- joint finger3_joint: axis 1 0 0 -> 0 1 0; limit lower=0.0 upper=0.01 effort=100 velocity=100 -> lower=-0.01 upper=0.0 effort=100 velocity=100; origin xyz=-0.03 0 -0.23 rpy=0 0 0 -> xyz=0 0.03 -0.23 rpy=0 0 0
- joint finger4_joint: axis 0 1 0 -> 1 0 0; origin xyz=0 -0.03 -0.23 rpy=0 0 0 -> xyz=-0.03 0 -0.23 rpy=0 0 0
- joint gripper_stretch: origin xyz=0.8 0 0 rpy=0 0 0 -> xyz=0 -0.8 0 rpy=0 0 0
- joint rotation2: origin xyz=1 0 0.1 rpy=0 0 0 -> xyz=0 -1 0.1 rpy=0 0 0

File: urdf/scara_robot_right.urdf (robot description, URDF)
Before this commit: robot scara_robot, 9 links, 8 joints
Links:
- link arm1: geometry collision box size=0.1 1.1 0.1; visual box size=0.1 1.1 0.1
- link arm2: geometry collision box size=0.1 0.9 0.1; visual box size=0.1 0.9 0.1
Joints:
- joint finger1_joint: axis 1 0 0 -> 0 1 0; origin xyz=0.03 0 -0.23 rpy=0 0 0 -> xyz=0 0.03 -0.23 rpy=0 0 0
- joint finger2_joint: axis 0 1 0 -> 1 0 0; limit lower=-0.01 upper=0.0 effort=100 velocity=100 -> lower=0.0 upper=0.01 effort=100 velocity=100; origin xyz=0 0.03 -0.23 rpy=0 0 0 -> xyz=-0.03 0 -0.23 rpy=0 0 0
- joint finger3_joint: axis 1 0 0 -> 0 1 0; origin xyz=-0.03 0 -0.23 rpy=0 0 0 -> xyz=0 -0.03 -0.23 rpy=0 0 0
- joint finger4_joint: axis 0 1 0 -> 1 0 0; limit lower=0.0 upper=0.01 effort=100 velocity=100 -> lower=-0.01 upper=0.0 effort=100 velocity=100; origin xyz=0 -0.03 -0.23 rpy=0 0 0 -> xyz=0.03 0 -0.23 rpy=0 0 0
- joint gripper_stretch: origin xyz=0.8 0 0 rpy=0 0 0 -> xyz=0 0.8 0 rpy=0 0 0
- joint rotation2: origin xyz=1 0 0.1 rpy=0 0 0 -> xyz=0 1 0.1 rpy=0 0 0

Commit message: update scara model

File: urdf/scara_robot_left.urdf (robot description, URDF)
Before this commit: robot scara_robot_left, 9 links, 8 joints
Joints:
- joint rotation2: limit lower=-3.13 upper=3.13 effort=100 velocity=100 -> lower=-3.00 upper=3.00 effort=100 velocity=100

File: urdf/scara_robot_right.urdf (robot description, URDF)
Before this commit: robot scara_robot_right, 9 links, 8 joints
Joints:
- joint rotation2: limit lower=-3.13 upper=3.13 effort=100 velocity=100 -> lower=-3.00 upper=3.00 effort=100 velocity=100

Commit message: finish gripper action server class def and implementation

File: urdf/scara_robot_left.urdf (robot description, URDF)
Before this commit: robot scara_robot_left, 9 links, 8 joints
Joints:
- removed joint gripper_stretch
- added joint gripper_joint: type prismatic, parent arm2, child gripper_link, origin xyz=0 -0.8 0 rpy=0 0 0, axis 0 0 1, limit lower=-0.05 upper=0.0 effort=100 velocity=100

File: urdf/scara_robot_right.urdf (robot description, URDF)
Before this commit: robot scara_robot_right, 9 links, 8 joints
Joints:
- removed joint gripper_stretch
- added joint gripper_joint: type prismatic, parent arm2, child gripper_link, origin xyz=0 0.8 0 rpy=0 0 0, axis 0 0 1, limit lower=-0.05 upper=0.0 effort=100 velocity=100

Commit message: finish all joint pd parameters tuning

File: urdf/scara_robot_left.urdf (robot description, URDF)
Before this commit: robot scara_robot_left, 9 links, 8 joints
Joints:
- joint rotation1: limit lower=-1.5708 upper=1.5708 effort=100 velocity=100 -> lower=-1.5708 upper=1.5708 effort=1000 velocity=1000
- joint rotation2: limit lower=-3.00 upper=3.00 effort=100 velocity=100 -> lower=-3.00 upper=3.00 effort=1000 velocity=1000

Commit message: increase joint 1 range in urdf

File: urdf/scara_robot_left.urdf (robot description, URDF)
Before this commit: robot scara_robot_left, 9 links, 8 joints
Joints:
- joint rotation1: limit lower=-1.5708 upper=1.5708 effort=1000 velocity=1000 -> lower=-2.6 upper=2.6 effort=1000 velocity=1000

File: urdf/scara_robot_right.urdf (robot description, URDF)
Before this commit: robot scara_robot_right, 9 links, 8 joints
Joints:
- joint rotation1: limit lower=-1.5708 upper=1.5708 effort=100 velocity=100 -> lower=-2.6 upper=2.6 effort=100 velocity=100

Commit message: one robot maneuver flow tuning

File: urdf/scara_robot_left.urdf (robot description, URDF)
Before this commit: robot scara_robot_left, 9 links, 8 joints
Joints:
- joint finger1_joint: limit lower=0.0 upper=0.01 effort=100 velocity=100 -> lower=0.0 upper=0.02 effort=100 velocity=100; origin xyz=0 -0.03 -0.23 rpy=0 0 0 -> xyz=0 -0.04 -0.23 rpy=0 0 0
- joint finger2_joint: limit lower=-0.01 upper=0.0 effort=100 velocity=100 -> lower=-0.02 upper=0.0 effort=100 velocity=100; origin xyz=0.03 0 -0.23 rpy=0 0 0 -> xyz=0.04 0 -0.23 rpy=0 0 0
- joint finger3_joint: limit lower=-0.01 upper=0.0 effort=100 velocity=100 -> lower=-0.02 upper=0.0 effort=100 velocity=100; origin xyz=0 0.03 -0.23 rpy=0 0 0 -> xyz=0 0.04 -0.23 rpy=0 0 0
- joint finger4_joint: limit lower=0.0 upper=0.01 effort=100 velocity=100 -> lower=0.0 upper=0.02 effort=100 velocity=100; origin xyz=-0.03 0 -0.23 rpy=0 0 0 -> xyz=-0.04 0 -0.23 rpy=0 0 0

File: urdf/scara_robot_right.urdf (robot description, URDF)
Before this commit: robot scara_robot_right, 9 links, 8 joints
Joints:
- joint finger1_joint: limit lower=-0.01 upper=0.0 effort=100 velocity=100 -> lower=-0.02 upper=0.0 effort=100 velocity=100; origin xyz=0 0.03 -0.23 rpy=0 0 0 -> xyz=0 0.04 -0.23 rpy=0 0 0
- joint finger2_joint: limit lower=0.0 upper=0.01 effort=100 velocity=100 -> lower=0.0 upper=0.02 effort=100 velocity=100; origin xyz=-0.03 0 -0.23 rpy=0 0 0 -> xyz=-0.04 0 -0.23 rpy=0 0 0
- joint finger3_joint: limit lower=0.0 upper=0.01 effort=100 velocity=100 -> lower=0.0 upper=0.02 effort=100 velocity=100; origin xyz=0 -0.03 -0.23 rpy=0 0 0 -> xyz=0 -0.04 -0.23 rpy=0 0 0
- joint finger4_joint: limit lower=-0.01 upper=0.0 effort=100 velocity=100 -> lower=-0.02 upper=0.0 effort=100 velocity=100; origin xyz=0.03 0 -0.23 rpy=0 0 0 -> xyz=0.04 0 -0.23 rpy=0 0 0

Commit message: finish motion parameter tuning

File: urdf/scara_robot_left.urdf (robot description, URDF)
Before this commit: robot scara_robot_left, 9 links, 8 joints
Links:
- link finger1: geometry collision box size=0.02 0.01 0.02; visual box size=0.02 0.01 0.02
- link finger2: geometry collision box size=0.01 0.02 0.02; visual box size=0.01 0.02 0.02
- link finger3: geometry collision box size=0.02 0.01 0.02; visual box size=0.02 0.01 0.02
- link finger4: geometry collision box size=0.01 0.02 0.02; visual box size=0.01 0.02 0.02

File: urdf/scara_robot_right.urdf (robot description, URDF)
Before this commit: robot scara_robot_right, 9 links, 8 joints
Links:
- link finger1: geometry collision box size=0.02 0.01 0.02; visual box size=0.02 0.01 0.02
- link finger2: geometry collision box size=0.01 0.02 0.02; visual box size=0.01 0.02 0.02
- link finger3: geometry collision box size=0.02 0.01 0.02; visual box size=0.02 0.01 0.02
- link finger4: geometry collision box size=0.01 0.02 0.02; visual box size=0.01 0.02 0.02
